File: hardware/V2.1.1/RP-Pico-Scope.kicad_sch (KiCad schematic)
At the start: 62 parts, among them J1 BNC-IN, Q1 BC547, Q2 BC557, Q3 C1815, Q4 BC547, Q5 BC557, U1 LM358, U2 NE555P, U3 TL084, U4 CD4052B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

Commit message: Update RP-Pico-Scope.kicad_sch
Connections:
- net -5VA: now also D5.2 (A)
- net GND: no longer D5.2 (A)
Changed lines of the file:
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@@
 		(company "by : HS6502")
 		(comment 1 "First Version Date : 17-Oct-2024")
-		(comment 2 "axiom + epsi1on")
 	)
 	(junction
@@
 	)
 	(junction
-		(at 113.03 105.41)
-		(diameter 0)
-		(color 0 0 0 0)
-	)
-	(junction
 		(at 88.9 92.71)
 		(diameter 0)
@@
 	(wire
 		(pts
-			(xy 125.73 105.41) (xy 113.03 105.41)
-		)
-		(stroke
-			(width 0)
-			(type default)
-		)
-	)
-	(wire
-		(pts
 			(xy 101.6 237.49) (xy 101.6 251.46)
 		)
@@
 					(unit 1)
 				)
+			)
+		)
+	)
+	(symbol
+		(lib_id "power:-5VA")
+		(at 125.73 105.41 180)
+		(unit 1)
+		(exclude_from_sim no)
+		(in_bom yes)
+		(on_board yes)
+		(dnp no)
+		(fields_autoplaced yes)
+		(property "Reference" "#PWR035"
+			(at 125.73 101.6 0)
+			(effects
+				(font
+					(size 1.27 1.27)
+				)
+				(hide yes)
+			)
+		)
+		(property "Value" "-5VA"
+			(at 125.73 110.49 0)
+			(effects
+				(font
+					(size 1.27 1.27)
+				)
+			)
+		)
+		(property "Footprint" ""
+			(at 125.73 105.41 0)
+			(effects
+				(font
+					(size 1.27 1.27)
+				)
+				(hide yes)
+			)
+		)
+		(property "Datasheet" ""
+			(at 125.73 105.41 0)
+			(effects
+				(font
+					(size 1.27 1.27)
+				)
+				(hide yes)
+			)
+		)
+		(property "Description" "Power symbol creates a global label with name \"-5VA\""
+			(at 125.73 105.41 0)
+			(effects
+				(font
+					(size 1.27 1.27)
+				)
+				(hide yes)
+			)
+		)
+		(pin "1"
+		)
+		(instances
+			(project "RP-Pico-Scope"
+				(path "/8d25a4ce-055a-4492-9644-c1eda4dd0215"
+					(reference "#PWR035")
+					(unit 1)
+				)
